Commit message: added gazebbo launch

File: urdf/accessories/wheel.xacro (robot description, xacro)
@@ -22,5 +22,5 @@
             </collision>
         </link>
-        <joint name="${wheel_prefix}_wheel" type="continuous">
+        <joint name="${wheel_prefix}_wheel_joint" type="continuous">
             <parent link="base_link"/>
             <child link="${wheel_prefix}_wheel_link"/>

File: urdf/basic_outdoor_robot.urdf.xacro (robot description, xacro)
@@ -27,4 +27,6 @@
     <!-- Dummy Values -->
     <xacro:property name="dummy_inertia" value="1e-09"/>
+    <!-- ros2 control params -->
+    <xacro:arg name="ros2_control_config" default="$(find basic_outdoor_robot_description)/config/control.yaml" />
     <!-- Base Link -->
     <link name="base_link">
@@ -53,7 +55,7 @@
     <link name="base_footprint"/>
     <joint name="base_footprint_joint" type="fixed">
-        <origin xyz="0 0 ${wheel_vertical_offset - wheel_radius}" rpy="0 0 0" />
-        <parent link="base_link" />
-        <child link="base_footprint" />
+        <origin xyz="0 0 ${-wheel_vertical_offset + wheel_radius}" rpy="0 0 0" />
+        <parent link="base_footprint" />
+        <child link="base_link" />
     </joint>
     <!-- Wheels -->
@@ -71,14 +73,11 @@
     </xacro:robot_wheel>
     <!-- IMU -->
-    <link name="imu_link">
-        <inertial>
-            <mass value="0.001"/>
-            <origin xyz="0 0 0" rpy="0 0 0"/>
-            <inertia ixx="${dummy_inertia}" ixy="0.0" ixz="0.0" iyy="${dummy_inertia}" iyz="0.0" izz="${dummy_inertia}"/>
-        </inertial>
-    </link>
     <joint name="imu_joint" type="fixed">
-        <parent link="base_link" />
+        <origin xyz="0 0 0" rpy="0 0 0" />
+        <parent link="base_link"/>
         <child link="imu_link" />
     </joint>
+    <link name="imu_link">
+    </link>
+    <xacro:include filename="$(find basic_outdoor_robot_description)/urdf/basic_outdoor_robot.gazebo" />
 </robot>
